Commit message: Minor model changes for fishbot

File: urdf/fishbot_simple.urdf.xacro (robot description, xacro)
@@ -15,5 +15,5 @@
         <child link="left_wheel_link"/>
         <axis rpy="0 0 0" xyz="0 1 0"/>
-        <origin xyz="0 0.023 -0.00925"/>
+        <origin xyz="0 0.023 -0.009"/>
     </joint>
     <joint name="right_wheel_joint" type="continuous">
@@ -21,5 +21,5 @@
         <child link="right_wheel_link"/>
         <axis rpy="0 0 0" xyz="0 1 0"/>
-        <origin xyz="0 -0.023 -0.00925"/>
+        <origin xyz="0 -0.023 -0.009"/>
     </joint>
     <joint name="support_1_joint" type="fixed">
